Commit message: added arm on dummy go1

File: resources/rx150-dummy-go1.urdf (robot description, URDF)
Before this commit: robot rx150, 12 links, 11 joints
Links:
- added link go1/base_link; collision box size=0.6 0.3 0.22; visual box size=0.6 0.3 0.22
- added link go1/fl_link; collision box size=0.05 0.05 0.25; visual box size=0.05 0.05 0.25
- added link go1/fr_link; collision box size=0.05 0.05 0.25; visual box size=0.05 0.05 0.25
- added link go1/rl_link; collision box size=0.05 0.05 0.25; visual box size=0.05 0.05 0.25
- added link go1/rr_link; collision box size=0.05 0.05 0.25; visual box size=0.05 0.05 0.25
Joints:
- added joint go1_arm_joint: type fixed, parent go1/base_link, child rx150/base_link, origin xyz=0.15 0 0.11 rpy=0 0 0, axis 1 0 0
- added joint go1_fl_joint: type fixed, parent go1/base_link, child go1/fl_link, origin xyz=0.25 0.1 -0.12 rpy=0 0 0, axis 1 0 0
- added joint go1_fr_joint: type fixed, parent go1/base_link, child go1/fr_link, origin xyz=0.25 -0.1 -0.12 rpy=0 0 0, axis 1 0 0
- added joint go1_rl_joint: type fixed, parent go1/base_link, child go1/rl_link, origin xyz=-0.25 0.1 -0.12 rpy=0 0 0, axis 1 0 0
- added joint go1_rr_joint: type fixed, parent go1/base_link, child go1/rr_link, origin xyz=-0.25 -0.1 -0.12 rpy=0 0 0, axis 1 0 0
